File: hbridge-proto.sch (KiCad schematic (older format))
At the start: 30 parts, among them IC1 LM5106, IC2 LM5106, J1 Screw_Terminal_1x03, J2 Screw_Terminal_1x02, J3 Screw_Terminal_1x02, J4 Screw_Terminal_1x02, Q1 TO-220-DUAL, Q2 TO-220-DUAL, Q3 TO-220-DUAL, Q4 TO-220-DUAL

Commit message: power trace layout
Parts:
- C1, C2, C3, C5, C6, R1, R10, R11, R2, R3, R4, R5, R6, R7, R8, R9: footprint (none) -> Resistors_SMD:R_0805_HandSoldering
- C4: footprint (none) -> Hbridge_proto:CAP_RADIAL_13MM
- D1, D2: footprint (none) -> Hbridge_proto:DO-214AC
- IC1, IC2: footprint (none) -> Housings_SSOP:MSOP-10_3x3mm_Pitch0.5mm
- J1: footprint (none) -> w_conn_mpt:mpt_0,5%2f3-2,54
- J2: footprint (none) -> w_conn_mpt:mpt_0,5%2f2-2,54
- J3, J4: footprint (none) -> Hbridge_proto:WURTH-2566-2
- Q1, Q2, Q3, Q4: footprint (none) -> Hbridge_proto:HEATSINK_TO-220_DUAL
- S1: footprint (none) -> Hbridge_proto:EG1218_SPDT
Connections:
- wire segments 86 -> 111

Commit message: first draft complete
Parts:
- renumbered Q4 to Q3, Q3 to Q4
Connections:
- wire segments 111 -> 86
Changed lines of the file:
@@
 $EndComp
 $Comp
-L TO-220-DUAL-RESCUE-hbridge-proto Q3
+L TO-220-DUAL-RESCUE-hbridge-proto Q4
 U 1 1 58D345BE
 P 7150 2250
-F 0 "Q3" H 7150 1450 60  0000 C CNN
+F 0 "Q4" H 7150 1450 60  0000 C CNN
 F 1 "TO-220-DUAL" H 7150 2250 60  0000 C CNN
 F 2 "Hbridge_proto:HEATSINK_TO-220_DUAL" H 7150 2250 60  0001 C CNN
@@
 $EndComp
 $Comp
-L TO-220-DUAL-RESCUE-hbridge-proto Q4
+L TO-220-DUAL-RESCUE-hbridge-proto Q3
 U 1 1 58D3466D
 P 7150 3600
-F 0 "Q4" H 7150 2800 60  0000 C CNN
+F 0 "Q3" H 7150 2800 60  0000 C CNN
 F 1 "TO-220-DUAL" H 7150 3600 60  0000 C CNN
 F 2 "Hbridge_proto:HEATSINK_TO-220_DUAL" H 7150 3600 60  0001 C CNN
@@
 $EndComp
 Wire Wire Line
-	5700 2400 6200 2400
-Wire Wire Line
-	6200 2400 6750 2400
+	5700 2400 6750 2400
 Wire Wire Line
 	6750 2400 6750 2500
@@
 	5700 2500 5700 2400
 Wire Wire Line
-	5800 1200 6200 1200
-Wire Wire Line
-	6200 1200 6500 1200
+	5800 1200 6500 1200
 Connection ~ 6500 1200
 Wire Wire Line
 	6500 1500 6500 1500
 Wire Wire Line
-	6200 1100 6200 1200
-Wire Wire Line
-	6200 1200 6200 2400
+	6200 1100 6200 2400
 Connection ~ 6200 1200
 Connection ~ 6200 2400
@@
 Connection ~ 6500 1500
 Wire Wire Line
-	5700 2800 5700 2900
-Wire Wire Line
-	5700 2900 5700 3400
-Wire Wire Line
-	5700 3400 5700 3750
-Wire Wire Line
-	5700 3750 5700 3850
-Wire Wire Line
-	6750 2800 6750 2900
-Wire Wire Line
-	6750 2900 6750 3400
-Wire Wire Line
-	6750 3400 6750 3750
-Wire Wire Line
-	6750 3750 6750 3850
+	5700 2800 5700 3850
+Wire Wire Line
+	6750 2800 6750 3850
 Wire Wire Line
 	5700 4150 5700 4250
@@
 Connection ~ 6750 2900
 Wire Wire Line
-	3900 3400 4350 3400
-Wire Wire Line
-	4350 3400 5700 3400
-Wire Wire Line
-	5700 3400 6100 3400
+	3900 3400 6100 3400
 Connection ~ 5700 3400
 Connection ~ 6750 3400
 Wire Wire Line
-	5700 4250 6200 4250
-Wire Wire Line
-	6200 4250 6750 4250
+	5700 4250 6750 4250
 Wire Wire Line
 	6200 4350 6200 4250
 Connection ~ 6200 4250
 Wire Wire Line
-	3900 3250 4000 3250
-Wire Wire Line
-	4000 3250 4050 3250
+	3900 3250 4050 3250
 Wire Wire Line
 	4000 3250 4000 2700
@@
 	2750 3250 3000 3250
 Wire Wire Line
-	3000 2550 3000 2700
-Wire Wire Line
-	3000 2700 3000 2950
-Wire Wire Line
-	3000 2950 3000 3100
+	3000 2550 3000 3100
 Wire Wire Line
 	3000 2950 2750 2950
@@
 	4550 2450 4500 2450
 Wire Wire Line
-	4500 2450 4500 2850
-Wire Wire Line
-	4500 2850 4500 3100
+	4500 2450 4500 3100
 Connection ~ 4500 3100
 Wire Wire Line
@@
 	4850 2850 4900 2850
 Wire Wire Line
-	4500 3550 4500 3800
-Wire Wire Line
-	4500 3800 4500 4200
+	4500 3550 4500 4200
 Wire Wire Line
 	4500 4200 4550 4200
@@
 	2200 3550 3000 3550
 Wire Wire Line
-	6300 3400 6750 3400
-Wire Wire Line
-	6750 3400 8150 3400
-Wire Wire Line
-	8150 3400 8600 3400
-Wire Wire Line
-	8450 3250 8500 3250
-Wire Wire Line
-	8500 3250 8600 3250
+	6300 3400 8600 3400
+Wire Wire Line
+	8450 3250 8600 3250
 Wire Wire Line
 	8500 3250 8500 2700
@@
 	9750 3250 9500 3250
 Wire Wire Line
-	9500 2550 9500 2700
-Wire Wire Line
-	9500 2700 9500 2950
-Wire Wire Line
-	9500 2950 9500 3100
+	9500 2550 9500 3100
 Wire Wire Line
 	9500 2950 9750 2950
@@
 	7950 2450 8000 2450
 Wire Wire Line
-	8000 2450 8000 2850
-Wire Wire Line
-	8000 2850 8000 3100
+	8000 2450 8000 3100
 Connection ~ 8000 3100
 Wire Wire Line
@@
 	7550 2850 7650 2850
 Wire Wire Line
-	8000 3550 8000 3800
-Wire Wire Line
-	8000 3800 8000 4200
+	8000 3550 8000 4200
 Wire Wire Line
 	8000 4200 7950 4200
@@
 	4900 5550 5000 5550
 Wire Wire Line
-	5300 5550 5400 5550
-Wire Wire Line
-	5400 5550 5800 5550
+	5300 5550 5800 5550
 Wire Wire Line
 	5400 5550 5400 5600

Commit message: via stitching
Parts:
- added TP? (x8): TEST, symbol TEST
Connections:
- wire segments 86 -> 87
Changed lines of the file:
@@
 	1    0    0    1
 $EndComp
+$Comp
+L TEST TP?
+U 1 1 58D39904
+P 4000 2700
+F 0 "TP?" H 4000 3000 50  0000 C BNN
+F 1 "TEST" H 4000 2950 50  0000 C CNN
+F 2 "" H 4000 2700 50  0000 C CNN
+F 3 "" H 4000 2700 50  0000 C CNN
+	1    4000 2700
+	1    0    0    -1
+$EndComp
+$Comp
+L TEST TP?
+U 1 1 58D39D09
+P 4500 2450
+F 0 "TP?" H 4500 2750 50  0000 C BNN
+F 1 "TEST" H 4500 2700 50  0000 C CNN
+F 2 "" H 4500 2450 50  0000 C CNN
+F 3 "" H 4500 2450 50  0000 C CNN
+	1    4500 2450
+	1    0    0    -1
+$EndComp
+$Comp
+L TEST TP?
+U 1 1 58D3A0A5
+P 4500 4200
+F 0 "TP?" H 4500 4500 50  0000 C BNN
+F 1 "TEST" H 4500 4450 50  0000 C CNN
+F 2 "" H 4500 4200 50  0000 C CNN
+F 3 "" H 4500 4200 50  0000 C CNN
+	1    4500 4200
+	-1   0    0    1
+$EndComp
+Wire Wire Line
+	2750 2950 2750 2800
+$Comp
+L TEST TP?
+U 1 1 58D3A645
+P 2750 2800
+F 0 "TP?" H 2750 3100 50  0000 C BNN
+F 1 "TEST" H 2750 3050 50  0000 C CNN
+F 2 "" H 2750 2800 50  0000 C CNN
+F 3 "" H 2750 2800 50  0000 C CNN
+	1    2750 2800
+	1    0    0    -1
+$EndComp
+$Comp
+L TEST TP?
+U 1 1 58D3B4DA
+P 8500 2700
+F 0 "TP?" H 8500 3000 50  0000 C BNN
+F 1 "TEST" H 8500 2950 50  0000 C CNN
+F 2 "" H 8500 2700 50  0000 C CNN
+F 3 "" H 8500 2700 50  0000 C CNN
+	1    8500 2700
+	1    0    0    -1
+$EndComp
+$Comp
+L TEST TP?
+U 1 1 58D3B79B
+P 9750 2950
+F 0 "TP?" H 9750 3250 50  0000 C BNN
+F 1 "TEST" H 9750 3200 50  0000 C CNN
+F 2 "" H 9750 2950 50  0000 C CNN
+F 3 "" H 9750 2950 50  0000 C CNN
+	1    9750 2950
+	1    0    0    -1
+$EndComp
+$Comp
+L TEST TP?
+U 1 1 58D3B849
+P 8000 2450
+F 0 "TP?" H 8000 2750 50  0000 C BNN
+F 1 "TEST" H 8000 2700 50  0000 C CNN
+F 2 "" H 8000 2450 50  0000 C CNN
+F 3 "" H 8000 2450 50  0000 C CNN
+	1    8000 2450
+	1    0    0    -1
+$EndComp
+$Comp
+L TEST TP?
+U 1 1 58D3B8DE
+P 8000 4200
+F 0 "TP?" H 8000 4500 50  0000 C BNN
+F 1 "TEST" H 8000 4450 50  0000 C CNN
+F 2 "" H 8000 4200 50  0000 C CNN
+F 3 "" H 8000 4200 50  0000 C CNN
+	1    8000 4200
+	-1   0    0    1
+$EndComp
 $EndSCHEMATC

Commit message: Improved driver signal routing
Parts:
- added R?: 0, Resistors_SMD:R_0805_HandSoldering, symbol R
- added TP9: TEST, Measurement_Points:Measurement_Point_Round-TH_Small, symbol TEST
- TP1, TP2, TP3, TP4, TP5, TP6, TP7, TP8: renamed from TP?; footprint (none) -> Measurement_Points:Measurement_Point_Round-SMD-Pad_Big
Connections:
- net labels added: DRV_2_IN_JMP
- wire segments 87 -> 88
Changed lines of the file:
@@
 	2000 1250 2000 1150
 Wire Wire Line
-	1850 1450 2000 1450
+	1850 1450 2300 1450
 Wire Wire Line
 	2000 1450 2000 1550
@@
 	1750 5300 2250 5300
 Wire Wire Line
-	1750 5500 2250 5500
+	1750 5500 2350 5500
 Wire Wire Line
 	1750 5700 1800 5700
@@
 $EndComp
 $Comp
-L TEST TP?
+L TEST TP2
 U 1 1 58D39904
 P 4000 2700
-F 0 "TP?" H 4000 3000 50  0000 C BNN
+F 0 "TP2" H 4000 3000 50  0000 C BNN
 F 1 "TEST" H 4000 2950 50  0000 C CNN
-F 2 "" H 4000 2700 50  0000 C CNN
+F 2 "Measurement_Points:Measurement_Point_Round-SMD-Pad_Big" H 4000 2700 50  0001 C CNN
 F 3 "" H 4000 2700 50  0000 C CNN
 	1    4000 2700
@@
 $EndComp
 $Comp
-L TEST TP?
+L TEST TP3
 U 1 1 58D39D09
 P 4500 2450
-F 0 "TP?" H 4500 2750 50  0000 C BNN
+F 0 "TP3" H 4500 2750 50  0000 C BNN
 F 1 "TEST" H 4500 2700 50  0000 C CNN
-F 2 "" H 4500 2450 50  0000 C CNN
+F 2 "Measurement_Points:Measurement_Point_Round-SMD-Pad_Big" H 4500 2450 50  0001 C CNN
 F 3 "" H 4500 2450 50  0000 C CNN
 	1    4500 2450
@@
 $EndComp
 $Comp
-L TEST TP?
+L TEST TP4
 U 1 1 58D3A0A5
 P 4500 4200
-F 0 "TP?" H 4500 4500 50  0000 C BNN
+F 0 "TP4" H 4500 4500 50  0000 C BNN
 F 1 "TEST" H 4500 4450 50  0000 C CNN
-F 2 "" H 4500 4200 50  0000 C CNN
+F 2 "Measurement_Points:Measurement_Point_Round-SMD-Pad_Big" H 4500 4200 50  0001 C CNN
 F 3 "" H 4500 4200 50  0000 C CNN
 	1    4500 4200
@@
 	2750 2950 2750 2800
 $Comp
-L TEST TP?
+L TEST TP1
 U 1 1 58D3A645
 P 2750 2800
-F 0 "TP?" H 2750 3100 50  0000 C BNN
+F 0 "TP1" H 2750 3100 50  0000 C BNN
 F 1 "TEST" H 2750 3050 50  0000 C CNN
-F 2 "" H 2750 2800 50  0000 C CNN
+F 2 "Measurement_Points:Measurement_Point_Round-SMD-Pad_Big" H 2750 2800 50  0001 C CNN
 F 3 "" H 2750 2800 50  0000 C CNN
 	1    2750 2800
@@
 $EndComp
 $Comp
-L TEST TP?
+L TEST TP7
 U 1 1 58D3B4DA
 P 8500 2700
-F 0 "TP?" H 8500 3000 50  0000 C BNN
+F 0 "TP7" H 8500 3000 50  0000 C BNN
 F 1 "TEST" H 8500 2950 50  0000 C CNN
-F 2 "" H 8500 2700 50  0000 C CNN
+F 2 "Measurement_Points:Measurement_Point_Round-SMD-Pad_Big" H 8500 2700 50  0001 C CNN
 F 3 "" H 8500 2700 50  0000 C CNN
 	1    8500 2700
@@
 $EndComp
 $Comp
-L TEST TP?
+L TEST TP8
 U 1 1 58D3B79B
 P 9750 2950
-F 0 "TP?" H 9750 3250 50  0000 C BNN
+F 0 "TP8" H 9750 3250 50  0000 C BNN
 F 1 "TEST" H 9750 3200 50  0000 C CNN
-F 2 "" H 9750 2950 50  0000 C CNN
+F 2 "Measurement_Points:Measurement_Point_Round-SMD-Pad_Big" H 9750 2950 50  0001 C CNN
 F 3 "" H 9750 2950 50  0000 C CNN
 	1    9750 2950
@@
 $EndComp
 $Comp
-L TEST TP?
+L TEST TP5
 U 1 1 58D3B849
 P 8000 2450
-F 0 "TP?" H 8000 2750 50  0000 C BNN
+F 0 "TP5" H 8000 2750 50  0000 C BNN
 F 1 "TEST" H 8000 2700 50  0000 C CNN
-F 2 "" H 8000 2450 50  0000 C CNN
+F 2 "Measurement_Points:Measurement_Point_Round-SMD-Pad_Big" H 8000 2450 50  0001 C CNN
 F 3 "" H 8000 2450 50  0000 C CNN
 	1    8000 2450
@@
 $EndComp
 $Comp
-L TEST TP?
+L TEST TP6
 U 1 1 58D3B8DE
 P 8000 4200
-F 0 "TP?" H 8000 4500 50  0000 C BNN
+F 0 "TP6" H 8000 4500 50  0000 C BNN
 F 1 "TEST" H 8000 4450 50  0000 C CNN
-F 2 "" H 8000 4200 50  0000 C CNN
+F 2 "Measurement_Points:Measurement_Point_Round-SMD-Pad_Big" H 8000 4200 50  0001 C CNN
 F 3 "" H 8000 4200 50  0000 C CNN
 	1    8000 4200
 	-1   0    0    1
 $EndComp
+$Comp
+L TEST TP9
+U 1 1 58D3C3AC
+P 2300 1450
+F 0 "TP9" H 2300 1750 50  0000 C BNN
+F 1 "TEST" H 2300 1700 50  0000 C CNN
+F 2 "Measurement_Points:Measurement_Point_Round-TH_Small" H 2300 1450 50  0001 C CNN
+F 3 "" H 2300 1450 50  0000 C CNN
+	1    2300 1450
+	1    0    0    -1
+$EndComp
+Connection ~ 2000 1450
+$Comp
+L R R?
+U 1 1 58D415D9
+P 2500 5500
+F 0 "R?" H 2600 5500 50  0000 C CNN
+F 1 "0" V 2500 5500 50  0000 C CNN
+F 2 "Resistors_SMD:R_0805_HandSoldering" V 2430 5500 50  0001 C CNN
+F 3 "" H 2500 5500 50  0000 C CNN
+	1    2500 5500
+	0    -1   -1   0
+$EndComp
+Wire Wire Line
+	2650 5500 2950 5500
+Text Label 2750 5500 0    60   ~ 0
+DRV_2_IN_JMP
 $EndSCHEMATC
